Commit message: update

File: sobit_edu_sim_description/robots/sobit_edu.urdf.xacro (robot description, xacro)
@@ -34,5 +34,5 @@
     <gazebo>
       <plugin name="gazebo_ros_control" filename="libgazebo_ros_control.so">
-        <robotNamespace>/$(arg robot_namespace)</robotNamespace>
+        <!-- <robotNamespace>/$(arg robot_namespace)</robotNamespace> -->
         <robotSimType>gazebo_ros_control/DefaultRobotHWSim</robotSimType>
         <legacyModeNS>true</legacyModeNS>

File: sobit_edu_sim_description/urdf/arm/arm.urdf.xacro (robot description, xacro)
@@ -14,20 +14,22 @@
         <origin xyz="0.0 0.0 0.0" rpy="0.0 0.0 ${M_PI/2.0}" />
         <geometry>
-          <mesh filename="package://sobit_edu_sim_description/meshes/arm/Assembly_2.stl" scale="1.0 1.0 1.0" />
+          <mesh filename="package://sobit_edu_sim_description/meshes/arm/arm_base.stl" scale="0.001 0.001 0.001" />
         </geometry>
         <material name="black" />
       </visual>
       <collision>
+        <!-- <origin xyz="0.0 0.01 0.0237" rpy="0.0 0.0 ${M_PI/2.0}" /> -->
         <origin xyz="0.0 0.0 0.0" rpy="0.0 0.0 ${M_PI/2.0}" />
         <geometry>
-          <mesh filename="package://sobit_edu_sim_description/meshes/arm/Assembly_2.stl" scale="1.0 1.0 1.0" />
+          <!-- <box size="0.06 0.06 0.0474"/> -->
+          <mesh filename="package://sobit_edu_sim_description/meshes/arm/arm_base.stl" scale="0.001 0.001 0.001" />
         </geometry>
       </collision>
       <inertial>
-        <origin xyz="0.0 0.0 0.0" rpy="0.0 0.0 0.0" />
-        <mass value="0.01" />
-        <inertia ixx="0.001" ixy="0.0" ixz="0.0"
-                 iyy="0.001" iyz="0.0"
-                 izz="0.001" />
+        <origin xyz="0.0 0.01 0.0237" rpy="0.0 0.0 0.0" />
+        <mass value="0.011" />
+        <inertia ixx="${1/12*0.011*(0.0474**2+0.06**2)}"  ixy="0.0" ixz="0.0"
+                 iyy="${1/12*0.011*(0.06**2+0.0474**2)}"  iyz="0.0"
+                 izz="${1/12*0.011*(0.06**2+0.06**2)}" />
       </inertial>
     </link>
@@ -43,20 +45,22 @@
         <origin xyz="0.0 0.0 0.0" rpy="0.0 0.0 ${M_PI/2.0}" />
         <geometry>
-          <mesh filename="package://sobit_edu_sim_description/meshes/arm/Assembly_3.stl" scale="1.0 1.0 1.0" />
+          <mesh filename="package://sobit_edu_sim_description/meshes/arm/arm_lower.stl" scale="0.001 0.001 0.001" />
         </geometry>
         <material name="black" />
       </visual>
       <collision>
+        <!-- <origin xyz="0.0 0.0 0.025875" rpy="0.0 0.0 ${M_PI/2.0}" /> -->
         <origin xyz="0.0 0.0 0.0" rpy="0.0 0.0 ${M_PI/2.0}" />
         <geometry>
-          <mesh filename="package://sobit_edu_sim_description/meshes/arm/Assembly_3.stl" scale="1.0 1.0 1.0" />
+          <!-- <box size="0.117 0.0285 0.05175"/> -->
+          <mesh filename="package://sobit_edu_sim_description/meshes/arm/arm_lower.stl" scale="0.001 0.001 0.001" />
         </geometry>
       </collision>
       <inertial>
-        <origin xyz="0.0 0.0 0.0" rpy="0.0 0.0 0.0" />
-        <mass value="0.01" />
-        <inertia ixx="0.001" ixy="0.0" ixz="0.0"
-                 iyy="0.001" iyz="0.0"
-                 izz="0.001" />
+        <origin xyz="0.0 0.0 0.0" rpy="0.0 0.0 0.025875" />
+        <mass value="0.023" />
+        <inertia ixx="${1/12*0.023*(0.05175**2+0.0285**2)}"  ixy="0.0" ixz="0.0"
+                 iyy="${1/12*0.023*(0.117**2+0.05175**2)}"  iyz="0.0"
+                 izz="${1/12*0.023*(0.117**2+0.0285**2)}" />
       </inertial>
     </link>
@@ -72,20 +76,21 @@
         <origin xyz="0 0.0 0.0" rpy="0.0 0.0 ${M_PI/2.0}" />
         <geometry>
-          <mesh filename="package://sobit_edu_sim_description/meshes/arm/Assembly_4.stl" scale="1.0 1.0  1.0 " />
+          <mesh filename="package://sobit_edu_sim_description/meshes/arm/arm_rotate.stl" scale="0.001 0.001 0.001" />
         </geometry>
         <material name="black" />
       </visual>
       <collision>
-        <origin xyz="0 0.0 0.0" rpy="0.0 0.0 ${M_PI/2.0}" />
+        <origin xyz="0.0 0.0 0.0" rpy="0.0 0.0 ${M_PI/2.0}" />
         <geometry>
-          <mesh filename="package://sobit_edu_sim_description/meshes/arm/Assembly_4.stl" scale="1.0  1.0  1.0 " />
+          <!-- <box size="0.117 0.1696 0.0475"/> -->
+          <mesh filename="package://sobit_edu_sim_description/meshes/arm/arm_rotate.stl" scale="0.001 0.001 0.001" />
         </geometry>
       </collision>
       <inertial>
         <origin xyz="0.0 0.0 0.0" rpy="0.0 0.0 0.0" />
-        <mass value="0.01" />
-        <inertia ixx="0.001" ixy="0.0" ixz="0.0"
-                 iyy="0.001" iyz="0.0"
-                 izz="0.001" />
+        <mass value="0.0179" />
+        <inertia ixx="${1/12*0.0179*(0.0475**2+0.1696**2)}"  ixy="0.0" ixz="0.0"
+                 iyy="${1/12*0.0179*(0.117**2+0.0475**2)}"  iyz="0.0"
+                 izz="${1/12*0.0179*(0.117**2+0.1696**2)}" />
       </inertial>
     </link>
@@ -110,5 +115,5 @@
         <origin xyz="0.0 0.0 0.0" rpy="0.0 0.0 ${M_PI/2.0}" />
         <geometry>
-          <mesh filename="package://sobit_edu_sim_description/meshes/arm/Assembly_5.stl" scale="1.0 1.0 1.0" />
+          <mesh filename="package://sobit_edu_sim_description/meshes/arm/arm_upper.stl" scale="0.001 0.001 0.001" />
         </geometry>
         <material name="black" />
@@ -117,13 +122,14 @@
         <origin xyz="0.0 0.0 0.0" rpy="0.0 0.0 ${M_PI/2.0}" />
         <geometry>
-          <mesh filename="package://sobit_edu_sim_description/meshes/arm/Assembly_5.stl" scale="1.0 1.0 1.0" />
+          <!-- <box size="0.0285 0.16375 0.0439"/> -->
+          <mesh filename="package://sobit_edu_sim_description/meshes/arm/arm_upper.stl" scale="0.001 0.001 0.001" />
         </geometry>
       </collision>
       <inertial>
         <origin xyz="0.0 0.0 0.0" rpy="0.0 0.0 ${M_PI/2.0}" />
-        <mass value="0.01" />
-        <inertia ixx="0.001" ixy="0.0" ixz="0.0"
-                 iyy="0.001" iyz="0.0"
-                 izz="0.001" />
+        <mass value="0.046" />
+        <inertia ixx="${1/12*0.046*(0.0475**2+0.1696**2)}"  ixy="0.0" ixz="0.0"
+                 iyy="${1/12*0.046*(0.117**2+0.0475**2)}"  iyz="0.0"
+                 izz="${1/12*0.046*(0.117**2+0.1696**2)}" />
       </inertial>
     </link>
@@ -146,5 +152,5 @@
     <link name="${prefix}_wrist_tilt_link" />
     <xacro:arm_transmission prefix="${prefix}" />
-    <xacro:arm_gazebo prefix="${prefix}"/>
+    <!-- <xacro:arm_gazebo prefix="${prefix}"/> -->
   </xacro:macro>
 </robot>

File: sobit_edu_sim_description/urdf/back/back.urdf.xacro (robot description, xacro)
@@ -18,4 +18,5 @@
         <origin xyz="0.0 0.0 0.0" rpy="0.0 0.0 ${M_PI/2}" />
         <geometry>
+          <!-- <box size="0.22703561 0.359 0.66023535"/> -->
           <mesh filename="package://sobit_edu_sim_description/meshes/back/back_base.stl" scale="0.001 0.001 0.001" />
         </geometry>
@@ -23,8 +24,8 @@
       <inertial>
         <origin xyz="0.0 0.0 0.0" rpy="0.0 0.0 0.0" />
-        <mass value="0.00004"/>
-        <inertia ixx="0.001" ixy="0.0" ixz="0.0"
-                 iyy="0.001" iyz="0.0"
-                 izz="0.001" />
+        <mass value="8.80" />
+        <inertia ixx="${1/12*8.80*(0.0474**2+0.66023535**2)}"  ixy="0.0" ixz="0.0"
+                 iyy="${1/12*8.80*(0.22703561**2+0.0474**2)}"  iyz="0.0"
+                 izz="${1/12*8.80*(0.22703561**2+0.66023535**2)}" />
       </inertial>
     </link>

File: sobit_edu_sim_description/urdf/base/base.urdf.xacro (robot description, xacro)
@@ -8,5 +8,5 @@
 <robot name="base" xmlns:xacro="http://ros.org/wiki/xacro">
   <xacro:include filename="$(find kobuki_description)/urdf/common_properties.urdf.xacro" />
-  <xacro:include filename="$(find kobuki_description)/urdf/kobuki_gazebo.urdf.xacro" />
+  <!-- <xacro:include filename="$(find kobuki_description)/urdf/kobuki_gazebo.urdf.xacro" /> -->
   <!-- Kobuki -->
   <xacro:macro name="base">
@@ -74,5 +74,5 @@
       </collision>
       <inertial>
-        <mass value="0.01" />
+        <mass value="10" />
         <origin xyz="0 0 0" />
         <inertia ixx="0.001" ixy="0.0" ixz="0.0"
@@ -101,5 +101,5 @@
       </collision>
       <inertial>
-        <mass value="0.01" />
+        <mass value="10" />
         <origin xyz="0 0 0" />
         <inertia ixx="0.001" ixy="0.0" ixz="0.0"
@@ -212,4 +212,14 @@
       <mu1>0.0</mu1>
       <mu2>0.0</mu2>
+    </gazebo>
+    <gazebo reference="wheel_l_link">
+	  <selfCollide>true</selfCollide>
+      <mu1>1.0</mu1>
+      <mu2>1.0</mu2>
+    </gazebo>
+    <gazebo reference="wheel_r_link">
+	  <selfCollide>true</selfCollide>
+      <mu1>1.0</mu1>
+      <mu2>1.0</mu2>
     </gazebo>
     <gazebo>

File: sobit_edu_sim_description/urdf/body/cover.urdf.xacro (robot description, xacro)
@@ -16,13 +16,17 @@
       </visual>
       <collision>
+        <!-- <origin xyz="-0.169875 0.0 -0.17239755" rpy="0.0 ${M_PI/2.0} ${-M_PI/2.0}" /> -->
         <origin xyz="0.0 0.0 0.0" rpy="0.0 ${M_PI/2.0} ${-M_PI/2.0}" />
         <geometry>
+          <!-- <box size="0.39853668 0.3447951 0.33975"/> -->
           <mesh filename="package://sobit_edu_sim_description/meshes/body/cover.stl" scale="0.001 0.001 0.001" />
         </geometry>
       </collision>
       <inertial>
-        <origin xyz="0.0 0.0 0.0" rpy="0.0 0.0 0.0" />
-        <mass value="1" />
-        <inertia ixx="0.0001" ixy="0.0" ixz="0.0" iyy="0.0001" iyz="0.0" izz="0.0001" />
+        <origin xyz="-0.169875 0.0 -0.17239755" rpy="0.0 ${M_PI/2.0} ${-M_PI/2.0}" />
+        <mass value="0.03" />
+        <inertia ixx="${1/12*0.03*(0.33975**2+0.3447951**2)}"  ixy="0.0" ixz="0.0"
+                 iyy="${1/12*0.03*(0.39853668**2+0.33975**2)}"  iyz="0.0"
+                 izz="${1/12*0.03*(0.39853668**2+0.3447951**2)}" />
       </inertial>
     </link>

File: sobit_edu_sim_description/urdf/body/stacks.urdf.xacro (robot description, xacro)
@@ -188,5 +188,6 @@
         <origin xyz="0.01364 0.0 0.0" rpy="0.0 0.0 0.0" />
         <geometry>
-          <mesh filename="package://turtlebot_description/meshes/stacks/hexagons/plate_simple.stl" scale="${M_SCALE} ${M_SCALE} ${M_SCALE}" />
+          <!-- <mesh filename="package://turtlebot_description/meshes/stacks/hexagons/plate_simple.stl" scale="${M_SCALE} ${M_SCALE} ${M_SCALE}" /> -->
+          <mesh filename="package://turtlebot_description/meshes/stacks/hexagons/plate_middle.dae" />
         </geometry>
       </collision>
@@ -221,5 +222,6 @@
         <origin xyz="0.01364 0.0 0.0" rpy="0.0 0.0 0.0" />
         <geometry>
-          <mesh filename="package://turtlebot_description/meshes/stacks/hexagons/plate_simple.stl" scale="${M_SCALE} ${M_SCALE} ${M_SCALE}" />
+          <!-- <mesh filename="package://turtlebot_description/meshes/stacks/hexagons/plate_simple.stl" scale="${M_SCALE} ${M_SCALE} ${M_SCALE}" /> -->
+          <mesh filename="package://turtlebot_description/meshes/stacks/hexagons/plate_top.dae" />
         </geometry>
       </collision>

File: sobit_edu_sim_description/urdf/hand/hand.gazebo.xacro (robot description, xacro)
@@ -7,40 +7,84 @@
       <mu2>1.0</mu2>
     </gazebo>
-    <gazebo reference="${prefix}_inner_l_link">
-      <selfCollide>false</selfCollide>
-      <mu1>1.0</mu1>
-      <mu2>1.0</mu2>
-    </gazebo>
-    <gazebo reference="${prefix}_inner_r_link">
-      <selfCollide>false</selfCollide>
-      <mu1>1.0</mu1>
-      <mu2>1.0</mu2>
-    </gazebo>
-    <gazebo reference="${prefix}_outer_l_link">
-      <selfCollide>false</selfCollide>
-      <mu1>1.0</mu1>
-      <mu2>1.0</mu2>
-    </gazebo>
-    <gazebo reference="${prefix}_outer_r_link">
-      <selfCollide>false</selfCollide>
-      <mu1>1.0</mu1>
-      <mu2>1.0</mu2>
-    </gazebo>
-    <gazebo reference="${prefix}_finger_l_link">
-      <selfCollide>false</selfCollide>
-      <mu1>1.0</mu1>
-      <mu2>1.0</mu2>
-    </gazebo>
-    <gazebo reference="${prefix}_finger_l_link">
-      <selfCollide>false</selfCollide>
-      <mu1>1.0</mu1>
-      <mu2>1.0</mu2>
-    </gazebo>
     <gazebo>
     <plugin name="joint_state_publisher" filename="libgazebo_ros_joint_state_publisher.so">
-      <jointName>hand_joint, hand_inner_l_joint, hand_finger_l_joint, hand_finger_r_joint, hand_outer_l_joint, hand_outer_r_joint</jointName>
+      <jointName>hand_joint</jointName>
       <updateRate>1000.0</updateRate>
     </plugin>
   </gazebo>
   </xacro:macro>
+  <xacro:macro name="mimic_joint" params="name_prefix parent_joint mimic_joint has_pid:=false multiplier:=1.0 offset:=0 sensitiveness:=0.0 max_effort:=1.0 robot_namespace:=''">
+    <gazebo>
+      <plugin name="${name_prefix}_mimic_joint_plugin" filename="libroboticsgroup_upatras_gazebo_mimic_joint_plugin.so">
+        <joint>${parent_joint}</joint>
+        <mimicJoint>${mimic_joint}</mimicJoint>
+        <xacro:if value="${has_pid}">                     <!-- if set to true, PID parameters from "/gazebo_ros_control/pid_gains/${mimic_joint}" are loaded -->
+          <hasPID />
+        </xacro:if>
+        <multiplier>${multiplier}</multiplier>
+        <offset>${offset}</offset>
+        <sensitiveness>${sensitiveness}</sensitiveness>   <!-- if absolute difference between setpoint and process value is below this threshold, do nothing; 0.0 = disable [rad] -->
+        <maxEffort>${max_effort}</maxEffort>              <!-- only taken into account if has_pid:=true [Nm] -->
+        <xacro:unless value="${robot_namespace == ''}">
+          <robotNamespace>${robot_namespace}</robotNamespace>
+        </xacro:unless>
+      </plugin>
+    </gazebo>
+  </xacro:macro>
+  <xacro:macro name="gazebo">
+    <!-- Gazebo -->
+    <gazebo>
+      <plugin name="gazebo_ros_control" filename="libgazebo_ros_control.so">
+        <robotNamespace>/$(arg robot_namespace)</robotNamespace>
+        <robotSimType>gazebo_ros_control/DefaultRobotHWSim</robotSimType>
+        <legacyModeNS>true</legacyModeNS>
+      </plugin>
+    </gazebo>
+    <!-- Mimic Joints -->
+    <xacro:mimic_joint
+      name_prefix="hand_inner_l_joint"
+      parent_joint="hand_joint"
+      mimic_joint="hand_inner_l_joint"
+      has_pid="false"
+      multiplier="1.0"
+      max_effort="10.0"
+      robot_namespace="$(arg robot_namespace)"
+    />
+    <xacro:mimic_joint
+      name_prefix="hand_outer_l_joint"
+      parent_joint="hand_inner_l_joint"
+      mimic_joint="hand_outer_l_joint"
+      has_pid="false"
+      multiplier="1.0"
+      max_effort="10.0"
+      robot_namespace="$(arg robot_namespace)"
+    />
+    <xacro:mimic_joint
+      name_prefix="hand_outer_r_joint"
+      parent_joint="hand_joint"
+      mimic_joint="hand_outer_r_joint"
+      has_pid="false"
+      multiplier="1.0"
+      max_effort="10.0"
+      robot_namespace="$(arg robot_namespace)"
+    />
+    <xacro:mimic_joint
+      name_prefix="hand_finger_l_joint"
+      parent_joint="hand_joint"
+      mimic_joint="hand_finger_l_joint"
+      has_pid="false"
+      multiplier="-1.0"
+      max_effort="10.0"
+      robot_namespace="$(arg robot_namespace)"
+    />
+    <xacro:mimic_joint
+      name_prefix="hand_finger_r_joint"
+      parent_joint="hand_joint"
+      mimic_joint="hand_finger_r_joint"
+      has_pid="false"
+      multiplier="-1.0"
+      max_effort="10.0"
+      robot_namespace="$(arg robot_namespace)"
+    />
+  </xacro:macro>
 </robot>

File: sobit_edu_sim_description/urdf/hand/hand.transmission.xacro (robot description, xacro)
@@ -4,4 +4,9 @@
   <xacro:macro name="hand_transmission" params="prefix_hand prefix_finger">
     <xacro:position_joint_transmission joint="${prefix_hand}_joint"         reduction="1" />
+    <!-- <xacro:position_joint_transmission joint="${prefix_hand}_inner_l_joint" reduction="1" />
+    <xacro:position_joint_transmission joint="${prefix_hand}_outer_l_joint" reduction="1" />
+    <xacro:position_joint_transmission joint="${prefix_hand}_outer_r_joint" reduction="1" />
+    <xacro:position_joint_transmission joint="${prefix_hand}_${prefix_finger}_l_joint" reduction="1" />
+    <xacro:position_joint_transmission joint="${prefix_hand}_${prefix_finger}_r_joint" reduction="1" /> -->
   </xacro:macro>
 </robot>

File: sobit_edu_sim_description/urdf/head/head.urdf.xacro (robot description, xacro)
@@ -18,15 +18,17 @@
       </visual>
       <collision>
+        <!-- <origin xyz="0.0 0.0077 0.00825" rpy="${M_PI/2.0} 0.0 ${M_PI/2.0}" /> -->
         <origin xyz="0.0 0.0 0.0" rpy="${M_PI/2.0} 0.0 ${M_PI/2.0}" />
         <geometry>
+          <!-- <box size="0.0285 0.0444 0.0905"/> -->
           <mesh filename="package://sobit_edu_sim_description/meshes/head/head_camera_base.stl" scale="0.001 0.001 0.001" />
         </geometry>
       </collision>
       <inertial>
-        <origin xyz="0.0 0.0 0.0" rpy="${M_PI/2.0} 0.0 ${M_PI/2.0}" />
-        <mass value="0.01" />
-        <inertia ixx="0.001" ixy="0.0" ixz="0.0"
-                 iyy="0.001" iyz="0.0"
-                 izz="0.001" />
+        <origin xyz="0.0 0.0077 0.00825" rpy="${M_PI/2.0} 0.0 ${M_PI/2.0}" />
+        <mass value="0.0014" />
+        <inertia ixx="${1/12*0.0014*(0.10471681**2+0.066**2)}"  ixy="0.0" ixz="0.0"
+                 iyy="${1/12*0.0014*(0.09414098**2+0.10471681**2)}"  iyz="0.0"
+                 izz="${1/12*0.0014*(0.09414098**2+0.066**2)}" />
       </inertial>
     </link>
@@ -47,15 +49,17 @@
       </visual>
       <collision>
+        <!-- <origin xyz="0.0005 0.0 0.027375" rpy="0.0 0.0 ${-M_PI/2.0}" /> -->
         <origin xyz="0.0 0.0 0.0" rpy="0.0 0.0 ${-M_PI/2.0}" />
         <geometry>
+          <!-- <box size="0.0454  0.0285 0.05475"/> -->
           <mesh filename="package://sobit_edu_sim_description/meshes/head/head_camera_pan.stl" scale="0.001 0.001 0.001" />
         </geometry>
       </collision>
       <inertial>
-        <origin xyz="0.0 0.0 0.0" rpy="0.0 0.0 ${-M_PI/2.0}" />
-        <mass value="0.01" />
-        <inertia ixx="0.001" ixy="0.0" ixz="0.0"
-                 iyy="0.001" iyz="0.0"
-                 izz="0.001" />
+        <origin xyz="0.0005 0.0 0.027375" rpy="0.0 0.0 ${-M_PI/2.0}" />
+        <mass value="0.0011" />
+        <inertia ixx="${1/12*0.0011*(0.05475**2+0.0285**2)}"  ixy="0.0" ixz="0.0"
+                 iyy="${1/12*0.0011*(0.0454**2+0.05475**2)}"  iyz="0.0"
+                 izz="${1/12*0.0011*(0.0454**2+0.0285**2)}" />
       </inertial>
     </link>
@@ -76,19 +80,21 @@
       </visual>
       <collision>
+        <!-- <origin xyz="0.0 0.0217 0.05626305" rpy="0.0 0.0 ${M_PI/2.0}" /> -->
         <origin xyz="0.0 0.0 0.0" rpy="0.0 0.0 ${M_PI/2.0}" />
         <geometry>
+          <!-- <box size="0.11640236 0.0994 0.1175261"/> -->
           <mesh filename="package://sobit_edu_sim_description/meshes/head/head_camera_tilt.stl" scale="0.001 0.001 0.001" />
         </geometry>
       </collision>
       <inertial>
-        <origin xyz="0.0 0.0 0.0" rpy="0.0 0.0 ${M_PI/2.0}" />
-        <mass value="0.01" />
-        <inertia ixx="0.001" ixy="0.0" ixz="0.0"
-                 iyy="0.001" iyz="0.0"
-                 izz="0.001" />
+        <origin xyz="0.0 0.0217 0.05626305" rpy="0.0 0.0 ${M_PI/2.0}" />
+        <mass value="0.0107" />
+        <inertia ixx="${1/12*0.0107*(0.1175261**2+0.0994**2)}"  ixy="0.0" ixz="0.0"
+                 iyy="${1/12*0.0107*(0.11640236**2+0.1175261**2)}"  iyz="0.0"
+                 izz="${1/12*0.0107*(0.11640236**2+0.0994**2)}" />
       </inertial>
     </link>
     <xacro:head_transmission prefix="${prefix}" />
-    <xacro:head_gazebo prefix="${prefix}" />
+    <!-- <xacro:head_gazebo prefix="${prefix}" /> -->
   </xacro:macro>
 </robot>

File: sobit_edu_sim_description/urdf/sensor/lidar.urdf.xacro (robot description, xacro)
@@ -16,15 +16,17 @@
       </visual>
       <collision>
+        <!-- <origin rpy="-0.05675 0.0 -0.0275" xyz="0.0 0.0 0.0" /> -->
         <origin rpy="0.0 0.0 ${M_PI}" xyz="0.0 0.0 0.0" />
         <geometry>
+          <!-- <box size="0.1575 0.05 0.055"/> -->
           <mesh filename="package://sobit_edu_sim_description/meshes/sensor/lidar_base.stl" scale="0.001 0.001 0.001" />
         </geometry>
       </collision>
       <inertial>
-        <origin rpy="0.0 0.0 0.0" xyz="0.0 0 0.0" />
-        <mass value="0.000001" />
-        <inertia ixx="0.0001" ixy="0.0" ixz="0.0"
-                 iyy="0.0001" iyz="0.0"
-                 izz="0.0001" />
+        <origin rpy="-0.05675 0.0 -0.0275" xyz="0.0 0.0 0.0" />
+        <mass value="0.35" />
+        <inertia ixx="${1/12*0.87*(0.055**2+0.05**2)}"  ixy="0.0" ixz="0.0"
+                 iyy="${1/12*0.87*(0.1575**2+0.055**2)}"  iyz="0.0"
+                 izz="${1/12*0.87*(0.1575**2+0.05**2)}" />
       </inertial>
     </link>

File: sobit_edu_sim_description/urdf/sensor/matrix.urdf.xacro (robot description, xacro)
@@ -20,4 +20,5 @@
         <origin xyz="0.0 0.0 0.0" rpy="0.0 0.0 0.0" />
         <geometry>
+          <!-- <box size="0.12419999 0.12419999 0.031758"/> -->
           <mesh filename="package://sobit_edu_sim_description/meshes/sensor/matrix_base.stl" scale="0.001 0.001 0.001" />
         </geometry>
@@ -25,8 +26,8 @@
       <inertial>
         <origin xyz="0.0 0.0 0.0" rpy="0.0 0.0 0.0" />
-        <mass value="1" />
-        <inertia ixx="0.001" ixy="0.0" ixz="0.0"
-                 iyy="0.001" iyz="0.0"
-                 izz="0.001" />
+        <mass value="0.078" />
+        <inertia ixx="${1/12*0.87*(0.12419999**2+0.031758**2)}"  ixy="0.0" ixz="0.0"
+                 iyy="${1/12*0.87*(0.12419999**2+0.12419999**2)}"  iyz="0.0"
+                 izz="${1/12*0.87*(0.12419999**2+0.031758**2)}" />
       </inertial>
     </link>
@@ -46,15 +47,17 @@
       </visual>
       <collision>
-        <origin xyz="0.0 0.0 0.0" rpy="0.0 0.0 0.0" />
+        <!-- <origin xyz="0.0 0.0 -0.0075" rpy="0.0 0.0 0.0" /> -->
+        <origin xyz="0.0 0.0 0.0" rpy="0.0 0.0 ${M_PI}" />
         <geometry>
+          <!-- <box size="0.10782796 0.10779832 0.0206"/> -->
           <mesh filename="package://sobit_edu_sim_description/meshes/sensor/matrix.stl" scale="0.001 0.001 0.001" />
         </geometry>
       </collision>
       <inertial>
-        <origin xyz="0.0 0.0 0.0" rpy="0.0 0.0 0.0" />
-        <mass value="1" />
-        <inertia ixx="0.001" ixy="0.0" ixz="0.0"
-                 iyy="0.001" iyz="0.0"
-                 izz="0.001" />
+        <origin xyz="0.0 0.0 -0.0075" rpy="0.0 0.0 0.0" />
+        <mass value="0.07" />
+        <inertia ixx="${1/12*0.87*(0.0206**2+0.10779832**2)}"  ixy="0.0" ixz="0.0"
+                 iyy="${1/12*0.87*(0.10782796**2+0.0206**2)}"  iyz="0.0"
+                 izz="${1/12*0.87*(0.10782796**2+0.10779832**2)}" />
       </inertial>
     </link>
