Commit message: update

File: sobit_edu_sim_description/urdf/sensor/mic.urdf.xacro (robot description, xacro)
@@ -18,4 +18,5 @@
         <origin xyz="0.0 0.0 0.0" rpy="${M_PI/2} 0 ${M_PI/2}" />
         <geometry>
+          <!-- <box size="0.02899298 0.03 0.03649824"/> -->
           <mesh filename="package://sobit_edu_sim_description/meshes/sensor/mic_base.stl" scale="0.001 0.001 0.001" />
         </geometry>
@@ -23,9 +24,9 @@
       </collision>
       <inertial>
-        <origin xyz="0.0 0.0 0.0" rpy="0 0 0" />
-        <mass value="1" />
-        <inertia ixx="0.001" ixy="0.0" ixz="0.0"
-                 iyy="0.001" iyz="0.0"
-                 izz="0.001" />
+        <origin xyz="0.0 0.0 0.0" rpy="${M_PI/2} 0 ${M_PI/2}" />
+        <mass value="0.02" />
+        <inertia ixx="${1/12*0.87*(0.03649824**2+0.03**2)}"  ixy="0.0" ixz="0.0"
+                 iyy="${1/12*0.87*(0.02899298**2+0.03649824**2)}"  iyz="0.0"
+                 izz="${1/12*0.87*(0.02899298**2+0.03**2)}" />
       </inertial>
     </link>
@@ -44,6 +45,8 @@
       </visual>
       <collision>
+        <!-- <origin xyz="0.0 0.02827923 -0.04872082" rpy="${M_PI} 0.0 ${M_PI/2}" /> -->
         <origin xyz="0.0 0.0 0.0" rpy="${M_PI} 0.0 ${M_PI/2}" />
         <geometry>
+          <!-- <box size="0.02999522 0.18154208 0.09744164"/> -->
           <mesh filename="package://sobit_edu_sim_description/meshes/sensor/mic.stl" scale="0.001 0.001 0.001" />
         </geometry>
@@ -51,9 +54,9 @@
       </collision>
       <inertial>
-        <origin xyz="0.0 0.0 0.0" rpy="0.0 0.0 0.0" />
-        <mass value="1" />
-        <inertia ixx="0.001" ixy="0.0" ixz="0.0"
-                 iyy="0.001" iyz="0.0"
-                 izz="0.001" />
+        <origin xyz="0.0 0.02827923 -0.04872082" rpy="${M_PI} 0.0 ${M_PI/2}" />
+        <mass value="0.47" />
+        <inertia ixx="${1/12*0.87*(0.09744164**2+0.18154208**2)}"  ixy="0.0" ixz="0.0"
+                 iyy="${1/12*0.87*(0.02999522**2+0.09744164**2)}"  iyz="0.0"
+                 izz="${1/12*0.87*(0.02999522**2+0.18154208**2)}" />
       </inertial>
     </link>
